File: hardware/TurbografxControllerToUSB.sch (KiCad schematic (older format))
At the start: 13 parts, among them CON1 AVR-ISP6, J1 USB, J2 DIN8, U1 ATMEGA32U2-AU, X1 16Mhz

Commit message: Slim down the board. Add footprind for mini-din8 on top of din8, this will allow to populate with both. Removing some kicad temp files.
Parts:
- added J3: MINIDIN8, symbol MINIDIN8
Connections:
- net labels added: DATA0, DATA1, DATA2, DATA3
- net labels removed: DOWN_SELECT_BUTTON, LEFT_RUN_BUTTON, RIGHT_II_BUTTON, UP_I_BUTTON
- wire segments 63 -> 75
Other:
- moved on the sheet: J2
Changed lines of the file:
@@
 LIBS:contrib
 LIBS:valves
+LIBS:conn_ext
 LIBS:TurbografxControllerToUSB-cache
 EELAYER 27 0
@@
 Sheet 1 1
 Title ""
-Date "5 aug 2014"
+Date "15 nov 2014"
 Rev ""
 Comp ""
@@
 SCK
 $Comp
-L GND #PWR09
-U 1 1 53DC1F3B
-P 9550 1150
-F 0 "#PWR09" H 9550 1150 30  0001 C CNN
-F 1 "GND" H 9550 1080 30  0001 C CNN
-F 2 "" H 9550 1150 60  0000 C CNN
-F 3 "" H 9550 1150 60  0000 C CNN
-	1    9550 1150
-	1    0    0    -1
-$EndComp
-Text GLabel 9700 1400 2    60   Input ~ 0
-DATA_SELECT
-Text GLabel 8150 1600 0    60   Input ~ 0
-RIGHT_II_BUTTON
-Text GLabel 9600 1750 2    60   Input ~ 0
-DOWN_SELECT_BUTTON
-$Comp
-L VCC #PWR010
+L VCC #PWR09
 U 1 1 53DC1FB2
-P 9650 1600
-F 0 "#PWR010" H 9650 1700 30  0001 C CNN
-F 1 "VCC" H 9650 1700 30  0000 C CNN
-F 2 "" H 9650 1600 60  0000 C CNN
-F 3 "" H 9650 1600 60  0000 C CNN
-	1    9650 1600
-	1    0    0    -1
-$EndComp
-Text GLabel 8350 1400 0    60   Input ~ 0
-~OE~
-Text GLabel 8150 1750 0    60   Input ~ 0
-LEFT_RUN_BUTTON
-Text GLabel 8150 1900 0    60   Input ~ 0
-UP_I_BUTTON
+P 9450 2450
+F 0 "#PWR09" H 9450 2550 30  0001 C CNN
+F 1 "VCC" H 9450 2550 30  0000 C CNN
+F 2 "" H 9450 2450 60  0000 C CNN
+F 3 "" H 9450 2450 60  0000 C CNN
+	1    9450 2450
+	1    0    0    -1
+$EndComp
 Text GLabel 4250 4800 0    60   Input ~ 0
 RESET
@@
 	2000 3750 2100 3750
 $Comp
-L GND #PWR011
+L GND #PWR010
 U 1 1 53DD24DF
 P 3750 3250
-F 0 "#PWR011" H 3750 3250 30  0001 C CNN
+F 0 "#PWR010" H 3750 3250 30  0001 C CNN
 F 1 "GND" H 3750 3180 30  0001 C CNN
 F 2 "" H 3750 3250 60  0000 C CNN
@@
 $EndComp
 $Comp
-L VCC #PWR012
+L VCC #PWR011
 U 1 1 53DD2647
 P 3750 2850
-F 0 "#PWR012" H 3750 2950 30  0001 C CNN
+F 0 "#PWR011" H 3750 2950 30  0001 C CNN
 F 1 "VCC" H 3750 2950 30  0000 C CNN
 F 2 "" H 3750 2850 60  0000 C CNN
@@
 $EndComp
 $Comp
-L GND #PWR013
+L GND #PWR012
 U 1 1 53DE7D12
 P 3950 2600
-F 0 "#PWR013" H 3950 2600 30  0001 C CNN
+F 0 "#PWR012" H 3950 2600 30  0001 C CNN
 F 1 "GND" H 3950 2530 30  0001 C CNN
 F 2 "" H 3950 2600 60  0000 C CNN
@@
 NoConn ~ 6700 3150
 $Comp
-L GND #PWR014
+L GND #PWR013
 U 1 1 53E0D3E1
-P 9350 1950
-F 0 "#PWR014" H 9350 1950 30  0001 C CNN
-F 1 "GND" H 9350 1880 30  0001 C CNN
-F 2 "" H 9350 1950 60  0000 C CNN
-F 3 "" H 9350 1950 60  0000 C CNN
-	1    9350 1950
+P 9600 2800
+F 0 "#PWR013" H 9600 2800 30  0001 C CNN
+F 1 "GND" H 9600 2730 30  0001 C CNN
+F 2 "" H 9600 2800 60  0000 C CNN
+F 3 "" H 9600 2800 60  0000 C CNN
+	1    9600 2800
 	1    0    0    -1
 $EndComp
@@
 L DIN8 J2
 U 1 1 53E0D96A
-P 8950 1550
-F 0 "J2" H 8950 1800 60  0000 C CNN
-F 1 "DIN8" H 8950 1100 60  0000 C CNN
-F 2 "~" H 8950 1550 60  0000 C CNN
-F 3 "~" H 8950 1550 60  0000 C CNN
-	1    8950 1550
-	1    0    0    -1
-$EndComp
-Wire Wire Line
-	8350 1400 8450 1400
-Wire Wire Line
-	8150 1600 8400 1600
-Wire Wire Line
-	9350 1300 9350 1100
-Wire Wire Line
-	9350 1100 9550 1100
-Wire Wire Line
-	9550 1100 9550 1150
-Wire Wire Line
-	9450 1400 9700 1400
-Wire Wire Line
-	9500 1600 9650 1600
-Wire Wire Line
-	9450 1700 9600 1700
-Wire Wire Line
-	9600 1700 9600 1750
-Wire Wire Line
-	9250 1850 9350 1850
-Wire Wire Line
-	9350 1850 9350 1950
-Wire Wire Line
-	8150 1750 8300 1750
-Wire Wire Line
-	8300 1750 8300 1700
-Wire Wire Line
-	8300 1700 8450 1700
-Wire Wire Line
-	8150 1900 8450 1900
-Wire Wire Line
-	8450 1900 8450 1800
-Wire Wire Line
-	8450 1800 8650 1800
+P 8750 2400
+F 0 "J2" H 8750 2650 60  0000 C CNN
+F 1 "DIN8" H 8750 1950 60  0000 C CNN
+F 2 "~" H 8750 2400 60  0000 C CNN
+F 3 "~" H 8750 2400 60  0000 C CNN
+	1    8750 2400
+	1    0    0    -1
+$EndComp
+Wire Wire Line
+	9300 2450 9450 2450
 Text GLabel 7000 4800 2    60   Input ~ 0
 ~OE~
-Text GLabel 7900 4900 2    60   Input ~ 0
-RIGHT_II_BUTTON
+Text GLabel 7400 4900 2    60   Input ~ 0
+DATA1
 Text GLabel 7000 5000 2    60   Input ~ 0
-LEFT_RUN_BUTTON
-Text GLabel 7900 5100 2    60   Input ~ 0
-UP_I_BUTTON
-Text GLabel 7900 5300 2    60   Input ~ 0
+DATA3
+Text GLabel 7400 5100 2    60   Input ~ 0
+DATA0
+Text GLabel 7400 5300 2    60   Input ~ 0
 DATA_SELECT
 Text GLabel 7000 5200 2    60   Input ~ 0
-DOWN_SELECT_BUTTON
+DATA2
 Wire Wire Line
 	6700 4800 7000 4800
@@
 	6700 5200 7000 5200
 NoConn ~ 6700 5400
-Wire Wire Line
-	6700 4900 7900 4900
-Wire Wire Line
-	6700 5100 7900 5100
-Wire Wire Line
-	6700 5300 7900 5300
+$Comp
+L MINIDIN8 J3
+U 1 1 5467B22D
+P 9400 4300
+F 0 "J3" H 9400 4600 60  0000 C CNN
+F 1 "MINIDIN8" H 9400 3950 60  0000 C CNN
+F 2 "" H 9400 4300 60  0000 C CNN
+F 3 "" H 9400 4300 60  0000 C CNN
+	1    9400 4300
+	1    0    0    -1
+$EndComp
+$Comp
+L GND #PWR014
+U 1 1 5467B2AF
+P 8900 4700
+F 0 "#PWR014" H 8900 4700 30  0001 C CNN
+F 1 "GND" H 8900 4630 30  0001 C CNN
+F 2 "" H 8900 4700 60  0000 C CNN
+F 3 "" H 8900 4700 60  0000 C CNN
+	1    8900 4700
+	1    0    0    -1
+$EndComp
+$Comp
+L VCC #PWR015
+U 1 1 5467B2B5
+P 10000 4600
+F 0 "#PWR015" H 10000 4700 30  0001 C CNN
+F 1 "VCC" H 10000 4700 30  0000 C CNN
+F 2 "" H 10000 4600 60  0000 C CNN
+F 3 "" H 10000 4600 60  0000 C CNN
+	1    10000 4600
+	1    0    0    -1
+$EndComp
+Wire Wire Line
+	9000 4550 8900 4550
+Wire Wire Line
+	8900 4150 8900 4700
+Wire Wire Line
+	9000 4150 8900 4150
+Connection ~ 8900 4550
+Wire Wire Line
+	9600 2150 9600 2800
+Wire Wire Line
+	9050 2700 9600 2700
+Connection ~ 9600 2700
+Wire Wire Line
+	9600 2150 9150 2150
+Wire Wire Line
+	9850 4450 9850 4600
+Wire Wire Line
+	9850 4600 10000 4600
+Wire Wire Line
+	9850 4350 10100 4350
+Wire Wire Line
+	9850 4250 10000 4250
+Wire Wire Line
+	10000 4250 10000 4200
+Wire Wire Line
+	10000 4200 10100 4200
+Wire Wire Line
+	9850 4150 9950 4150
+Wire Wire Line
+	9950 4150 9950 4050
+Wire Wire Line
+	9950 4050 10100 4050
+Wire Wire Line
+	9000 4050 8800 4050
+Wire Wire Line
+	9000 4250 8800 4250
+Wire Wire Line
+	9000 4350 9000 4400
+Wire Wire Line
+	9000 4400 8800 4400
+Wire Wire Line
+	8250 2250 8100 2250
+Wire Wire Line
+	8200 2450 8200 2400
+Wire Wire Line
+	8200 2400 8100 2400
+Wire Wire Line
+	8250 2550 8100 2550
+Wire Wire Line
+	8450 2650 8200 2650
+Wire Wire Line
+	8200 2650 8200 2700
+Wire Wire Line
+	8200 2700 8100 2700
+Wire Wire Line
+	9250 2250 9650 2250
+Wire Wire Line
+	9250 2550 9650 2550
+Wire Wire Line
+	7400 4900 6700 4900
+Wire Wire Line
+	7400 5100 6700 5100
+Wire Wire Line
+	7400 5300 6700 5300
+Text GLabel 8800 4400 0    60   Input ~ 0
+DATA0
+Text GLabel 8100 2700 0    60   Input ~ 0
+DATA0
+Text GLabel 10100 4200 2    60   Input ~ 0
+DATA1
+Text GLabel 8100 2400 0    60   Input ~ 0
+DATA1
+Text GLabel 10100 4350 2    60   Input ~ 0
+DATA2
+Text GLabel 9650 2550 2    60   Input ~ 0
+DATA2
+Text GLabel 8800 4250 0    60   Input ~ 0
+DATA3
+Text GLabel 8100 2550 0    60   Input ~ 0
+DATA3
+Text GLabel 10100 4050 2    60   Input ~ 0
+DATA_SELECT
+Text GLabel 9650 2250 2    60   Input ~ 0
+DATA_SELECT
+Text GLabel 8800 4050 0    60   Input ~ 0
+~OE~
+Text GLabel 8100 2250 0    60   Input ~ 0
+~OE~
 $EndSCHEMATC
